File: feasibility_prototypes/ir_board/feas_prot_ir_board.sch (KiCad schematic (older format))
At the start: 10 parts, among them P1 CONN_01X04, P2 CONN_01X04, P3 CONN_02X08, P4 CONN_02X08, Q1 APT2012P3BT

Commit message: Added RJ11 connector to processor board, finished IR board.
Parts:
- P1: footprint (none) -> med_conn_prototype_footprints:Sullins_SMD_pin_header_1x4_GBC36SABN-M30
- P2: footprint (none) -> med_conn_prototype_footprints:wire_solder_pad_2.54mm_1x4
Changed lines of the file:
@@
 $EndComp
 $Comp
-L GND #PWR1
+L GND #PWR01
 U 1 1 58ADC222
 P 4000 4000
-F 0 "#PWR1" H 4000 3750 50  0001 C CNN
+F 0 "#PWR01" H 4000 3750 50  0001 C CNN
 F 1 "GND" H 4000 3850 50  0000 C CNN
 F 2 "" H 4000 4000 50  0000 C CNN
@@
 $EndComp
 $Comp
-L GND #PWR3
+L GND #PWR02
 U 1 1 58ADC242
 P 4750 4000
-F 0 "#PWR3" H 4750 3750 50  0001 C CNN
+F 0 "#PWR02" H 4750 3750 50  0001 C CNN
 F 1 "GND" H 4750 3850 50  0000 C CNN
 F 2 "" H 4750 4000 50  0000 C CNN
@@
 F 0 "P2" H 4700 1850 50  0000 C CNN
 F 1 "CONN_01X04" H 4750 1350 50  0000 C CNN
-F 2 "" H 4700 1600 50  0000 C CNN
+F 2 "med_conn_prototype_footprints:wire_solder_pad_2.54mm_1x4" H 4700 1600 50  0001 C CNN
 F 3 "" H 4700 1600 50  0000 C CNN
 	1    4700 1600
@@
 F 0 "P1" H 4700 2200 50  0000 C CNN
 F 1 "CONN_01X04" H 4550 1700 50  0000 C CNN
-F 2 "" H 4700 1950 50  0000 C CNN
+F 2 "med_conn_prototype_footprints:Sullins_SMD_pin_header_1x4_GBC36SABN-M30" H 4700 1950 50  0001 C CNN
 F 3 "" H 4700 1950 50  0000 C CNN
 	1    4700 1950
@@
 	4550 2400 4450 2400
 $Comp
-L GND #PWR2
+L GND #PWR03
 U 1 1 58AEB5B1
 P 4450 2400
-F 0 "#PWR2" H 4450 2150 50  0001 C CNN
+F 0 "#PWR03" H 4450 2150 50  0001 C CNN
 F 1 "GND" H 4450 2250 50  0000 C CNN
 F 2 "" H 4450 2400 50  0000 C CNN
