File: feasibility_circuits/ldo_regulator_modules/s-1206_based_2V_regulator/rev.1/s-1206_based_2V_regulator.kicad_pcb (KiCad board)
At the start: 2 copper layers, 139.7 x 33 mm, 32 parts, among them J1 Jumper, J2 Jumper, J3 Jumper, J4 Jumper, J5 Jumper, J6 Jumper, P1 VIN, P10 TEST_VOUT_1_2, P11 TEST_VOUT_2_2, P12 TEST_VOUT_3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

Commit message: Updated gerber generation settings for battery and LDO test boards
Routing:
- net GND: vias 10 -> 0
- net (no net): vias 0 -> 10
Changed lines of the file:
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@@
   (general
     (links 43)
-    (no_connects 2)
+    (no_connects 5)
     (area 88.824999 87.554999 228.675001 120.725001)
     (thickness 1.6)
@@
     (visible_elements 7FFFFFFF)
     (pcbplotparams
-      (layerselection 0x00030_80000001)
+      (layerselection 0x01000_80000001)
       (usegerberextensions false)
       (excludeedgelayer true)
@@
       (outputformat 1)
       (mirror false)
-      (drillshape 1)
+      (drillshape 0)
       (scaleselection 1)
-      (outputdirectory ""))
+      (outputdirectory gerber/))
   )
   (net 0 "")
@@
   (gr_line (start 88.9 88.9) (end 88.9 87.63) (angle 90) (layer Edge.Cuts) (width 0.15))
   (gr_line (start 88.9 104.14) (end 88.9 88.9) (angle 90) (layer Edge.Cuts) (width 0.15))
+  (via (at 149.86 90.17) (size 1.5) (drill 0.7) (layers F.Cu B.Cu) (net 0))
+  (via (at 149.86 118.11) (size 1.5) (drill 0.7) (layers F.Cu B.Cu) (net 0))
+  (via (at 198.12 114.3) (size 1.5) (drill 0.7) (layers F.Cu B.Cu) (net 0))
+  (via (at 198.12 93.98) (size 1.5) (drill 0.7) (layers F.Cu B.Cu) (net 0))
+  (via (at 109.22 110.49) (size 1.5) (drill 0.7) (layers F.Cu B.Cu) (net 0))
+  (via (at 109.22 97.79) (size 1.5) (drill 0.7) (layers F.Cu B.Cu) (net 0))
+  (via (at 162.56 105.41) (size 1.5) (drill 0.7) (layers F.Cu B.Cu) (net 0))
+  (via (at 137.16 105.41) (size 1.5) (drill 0.7) (layers F.Cu B.Cu) (net 0))
+  (via (at 149.86 113.03) (size 1.5) (drill 0.7) (layers F.Cu B.Cu) (net 0))
+  (via (at 149.86 105.41) (size 1.5) (drill 0.7) (layers F.Cu B.Cu) (net 0))
   (segment (start 148.92 109.22) (end 150.8 109.22) (width 0.3) (layer F.Cu) (net 1))
   (segment (start 148.92 109.22) (end 147.32 109.22) (width 0.3) (layer F.Cu) (net 1))
@@
   (segment (start 130.81 107.95) (end 133.37 110.51) (width 1) (layer F.Cu) (net 1))
   (segment (start 127.02 107.95) (end 127.02 107.97) (width 1) (layer F.Cu) (net 1))
-  (via (at 149.86 90.17) (size 1.5) (drill 0.7) (layers F.Cu B.Cu) (net 2))
-  (via (at 149.86 118.11) (size 1.5) (drill 0.7) (layers F.Cu B.Cu) (net 2))
-  (via (at 198.12 114.3) (size 1.5) (drill 0.7) (layers F.Cu B.Cu) (net 2))
-  (via (at 198.12 93.98) (size 1.5) (drill 0.7) (layers F.Cu B.Cu) (net 2))
-  (via (at 109.22 110.49) (size 1.5) (drill 0.7) (layers F.Cu B.Cu) (net 2))
-  (via (at 109.22 97.79) (size 1.5) (drill 0.7) (layers F.Cu B.Cu) (net 2))
-  (via (at 162.56 105.41) (size 1.5) (drill 0.7) (layers F.Cu B.Cu) (net 2))
-  (via (at 137.16 105.41) (size 1.5) (drill 0.7) (layers F.Cu B.Cu) (net 2))
-  (via (at 149.86 113.03) (size 1.5) (drill 0.7) (layers F.Cu B.Cu) (net 2))
-  (via (at 149.86 105.41) (size 1.5) (drill 0.7) (layers F.Cu B.Cu) (net 2))
   (segment (start 151.16 96.84) (end 153.37 96.84) (width 1) (layer F.Cu) (net 2))
   (segment (start 153.37 96.84) (end 153.67 96.54) (width 1) (layer F.Cu) (net 2))
