File: feasibility_circuits/constant_current_load_modules/four_constant_current_loads/rev.1/four_constant_current_loads.sch (KiCad schematic (older format))
At the start: 96 parts

Commit message: Completed layout of constant current load PCB, the zip file sent for production is also included
Parts:
- D1, D2, D3, D4: renamed from D?; symbol LED -> LED-RESCUE-four_constant_current_loads
- gave numbers to parts that had none: 92
